File: opticalAbsorptionMeasurement.kicad_sch (KiCad schematic)
At the start: 131 parts, among them J1 Conn_01x02_Male, J2 Conn_01x02_Male, J3 Conn_01x03_Male, J4 Conn_01x03_Male, J5 Conn_01x03_Male, J6 Conn_01x03_Male, J7 Conn_01x02_Male, J8 Conn_01x02_Male, J9 Conn_01x02_Male, Q1 J111, Q2 J111, Q3 J111, Q4 J111, U1 TEN5-0523, U10 ADR01, U11 OPA602AU, U12 OPA602AU, U13 OPA602AU, U14 OPA602AU, U15 OPA602AU, U16 OPA602AU, U19 OPA602AU, U2 OPA602AU, U20 OPA602AU, U21 OPA602AU, U22 OPA602AU, U23 OPA602AU, U24 OPA602AU, U3 OPA602AU, U6 L7812, U7 L7912, U8 OPA602AU, U9 OPA602AU

Commit message: update resistor
update resistor
Parts:
- added R39, R40: 10k, Resistor_THT:R_Axial_DIN0207_L6.3mm_D2.5mm_P10.16mm_Horizontal, symbol Device:R
Connections:
- net +15V: now also R39.2
- net -15V: now also R40.1
- net GND: now also R39.1, R40.2
Changed lines of the file:
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@@
   (junction (at 135.89 63.5) (diameter 0) (color 0 0 0 0)
   )
+  (junction (at 38.1 33.02) (diameter 0) (color 0 0 0 0)
+  )
   (junction (at 374.65 179.07) (diameter 0) (color 0 0 0 0)
   )
@@
     (stroke (width 0) (type default) (color 0 0 0 0))
   )
+  (wire (pts (xy 38.1 24.13) (xy 49.53 24.13))
+    (stroke (width 0) (type default) (color 0 0 0 0))
+  )
   (wire (pts (xy 213.36 129.54) (xy 217.17 129.54))
     (stroke (width 0) (type default) (color 0 0 0 0))
@@
     (stroke (width 0) (type default) (color 0 0 0 0))
   )
+  (wire (pts (xy 38.1 41.91) (xy 49.53 41.91))
+    (stroke (width 0) (type default) (color 0 0 0 0))
+  )
   (wire (pts (xy 114.3 133.35) (xy 114.3 135.89))
     (stroke (width 0) (type default) (color 0 0 0 0))
@@
     (stroke (width 0) (type default) (color 0 0 0 0))
   )
+  (wire (pts (xy 38.1 40.64) (xy 38.1 41.91))
+    (stroke (width 0) (type default) (color 0 0 0 0))
+  )
   (wire (pts (xy 125.73 218.44) (xy 124.46 218.44))
     (stroke (width 0) (type default) (color 0 0 0 0))
@@
     (stroke (width 0) (type default) (color 0 0 0 0))
   )
+  (wire (pts (xy 38.1 31.75) (xy 38.1 33.02))
+    (stroke (width 0) (type default) (color 0 0 0 0))
+  )
   (wire (pts (xy 140.97 129.54) (xy 144.78 129.54))
     (stroke (width 0) (type default) (color 0 0 0 0))
@@
     (stroke (width 0) (type default) (color 0 0 0 0))
   )
+  (wire (pts (xy 38.1 33.02) (xy 49.53 33.02))
+    (stroke (width 0) (type default) (color 0 0 0 0))
+  )
   (wire (pts (xy 292.1 215.9) (xy 292.1 219.71))
     (stroke (width 0) (type default) (color 0 0 0 0))
@@
     (pin "1")
   )
+  (symbol (lib_id "Device:R") (at 38.1 27.94 180) (unit 1)
+    (in_bom yes) (on_board yes)
+    (property "Reference" "R39" (id 0) (at 34.29 31.75 90))
+    (property "Value" "10k" (id 1) (at 34.29 27.94 90))
+    (property "Footprint" "Resistor_THT:R_Axial_DIN0207_L6.3mm_D2.5mm_P10.16mm_Horizontal" (id 2) (at 39.878 27.94 90)
+      (effects (font (size 1.27 1.27)) hide)
+    )
+    (property "Datasheet" "~" (id 3) (at 38.1 27.94 0)
+      (effects (font (size 1.27 1.27)) hide)
+    )
+    (pin "1")
+    (pin "2")
+  )
   (symbol (lib_id "Device:C") (at 198.12 201.93 90) (unit 1)
     (in_bom yes) (on_board yes) (fields_autoplaced)
@@
     (pin "1")
   )
+  (symbol (lib_id "Device:R") (at 38.1 36.83 180) (unit 1)
+    (in_bom yes) (on_board yes)
+    (property "Reference" "R40" (id 0) (at 34.29 40.64 90))
+    (property "Value" "10k" (id 1) (at 34.29 36.83 90))
+    (property "Footprint" "Resistor_THT:R_Axial_DIN0207_L6.3mm_D2.5mm_P10.16mm_Horizontal" (id 2) (at 39.878 36.83 90)
+      (effects (font (size 1.27 1.27)) hide)
+    )
+    (property "Datasheet" "~" (id 3) (at 38.1 36.83 0)
+      (effects (font (size 1.27 1.27)) hide)
+    )
+    (pin "1")
+    (pin "2")
+  )
   (symbol (lib_id "Device:R") (at 120.65 207.01 90) (unit 1)
     (in_bom yes) (on_board yes) (fields_autoplaced)
@@
       (reference "R38") (unit 1) (value "1M") (footprint "Resistor_THT:R_Axial_DIN0207_L6.3mm_D2.5mm_P10.16mm_Horizontal")
     )
+    (path "/6ea8b656-f095-40d8-83da-4420a347720c"
+      (reference "R39") (unit 1) (value "10k") (footprint "Resistor_THT:R_Axial_DIN0207_L6.3mm_D2.5mm_P10.16mm_Horizontal")
+    )
+    (path "/8ab8b2fe-1bb9-431a-8ae3-9c8b3fbf62f6"
+      (reference "R40") (unit 1) (value "10k") (footprint "Resistor_THT:R_Axial_DIN0207_L6.3mm_D2.5mm_P10.16mm_Horizontal")
+    )
     (path "/26d156b9-6846-4c70-bc14-132913353f59"

Commit message: bom list
Other:
- company: (none) -> elektrotechnik2go.de
Changed lines of the file:
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@@
   (title_block
     (title "opticalAbsorptionMeasurement")
-    (date "2022-11-17")
-    (rev "1.0")
+    (date "2023-05-11")
+    (rev "1.1")
+    (company "elektrotechnik2go.de")
+    (comment 1 "Johann Schmid")
   )
   (junction (at 135.89 50.8) (diameter 0) (color 0 0 0 0)
